Commit message: added base stl file!

File: Fun_Projects/RJJE_Arm/rjje_arm_ws/src/rjje_arm/urdf/definitions.xacro (robot description, xacro)
@@ -1,4 +1,10 @@
 <?xml version="1.0"?>
-<robot name="rjje_arm" xmlns:xacro="http://www.ros.org/wiki/xacro">
+<robot name="definitions" xmlns:xacro="http://www.ros.org/wiki/xacro">
+  <material name="blue">
+    <color rgba="0 0 0.8 1"/>
+  </material>
+  <material name="light_black">
+    <color rgba="0.2 0.2 0.1 1.0"/>
+  </material>
   <xacro:macro name="m_link_mesh" params="name origin_xyz origin_rpy meshfile meshscale mass ixx ixy ixz iyy iyz izz">
     <link name="${name}">
@@ -32,22 +38,3 @@
     </joint>
   </xacro:macro>
-  <!-- Instances -->
-  <link name="world">
-  </link>
-  <xacro:m_link_mesh
-    name="base_link"
-    origin_xyz="0.0 0.0 0.0"
-    origin_rpy="0.0 0.0 0.0"
-    meshfile="package://rjje_arm/meshes/cup_holder.stl"
-    meshscale="0.1 0.1 0.1"
-    mass="157.633"
-    ixx="13.235" ixy="0" ixz="0"
-    iyy="13.235" iyz="0"
-    izz="9.655"
-    />
-  <xacro:m_joint name="$base_link_world" type="revolute"
-         axis_xyz="0 0 1"
-         origin_rpy="0 0 0" origin_xyz="0 0 0.0"
-         parent="world" child="base_link"
-         limit_e="1000" limit_l="0" limit_u="0.5" limit_v="0.5" />
 </robot>

File: Fun_Projects/RJJE_Arm/rjje_arm_ws/src/rjje_arm/urdf/rjje_arm.xacro.urdf (robot description, URDF)
Before this commit: robot rjje_arm, 2 links, 1 joints
Links:
- link base_link: geometry collision mesh filename=package://rjje_arm/meshes/base.stl scale=0.1 0.1 0.1; visual mesh filename=package://rjje_arm/meshes/base.stl scale=0.1 0.1 0.1

Commit message: added first real link!

File: Fun_Projects/RJJE_Arm/rjje_arm_ws/src/rjje_arm/urdf/definitions.xacro (robot description, xacro)
@@ -4,8 +4,11 @@
     <color rgba="0 0 0.8 1"/>
   </material>
-  <material name="light_black">
+  <material name="yellow">
+    <color rgba="0.93 0.93 0.02 1.0"/>
+  </material>
+  <material name="dark_green">
     <color rgba="0.2 0.2 0.1 1.0"/>
   </material>
-  <xacro:macro name="m_link_mesh" params="name origin_xyz origin_rpy meshfile meshscale mass ixx ixy ixz iyy iyz izz">
+  <xacro:macro name="m_link_mesh" params="name origin_xyz origin_rpy meshfile meshscale mass ixx ixy ixz iyy iyz izz color">
     <link name="${name}">
       <inertial>
@@ -25,10 +28,10 @@
           <mesh filename="${meshfile}" scale="${meshscale}"/>
         </geometry>
-        <material name="light_black"/>
+        <material name="${color}"/>
       </visual>
     </link>
   </xacro:macro>
-  <xacro:macro name="m_joint" params="name type axis_xyz origin_rpy origin_xyz parent child limit_e limit_l limit_u limit_v">
-    <joint name="${name}" type="${type}">
+  <xacro:macro name="m_joint" params="type axis_xyz origin_rpy origin_xyz parent child limit_e limit_l limit_u limit_v">
+    <joint name="${parent}_${child}" type="${type}">
       <axis xyz="${axis_xyz}"/>
       <limit effort="${limit_e}" lower="${limit_l}" upper="${limit_u}" velocity="${limit_v}" />

File: Fun_Projects/RJJE_Arm/rjje_arm_ws/src/rjje_arm/urdf/rjje_arm.xacro (robot description, xacro)
@@ -10,14 +10,49 @@
     origin_rpy="0.0 0.0 0.0"
     meshfile="package://rjje_arm/meshes/base.stl"
-    meshscale="0.1 0.1 0.1"
+    meshscale="1 1 1"
     mass="157.633"
     ixx="13.235" ixy="0" ixz="0"
     iyy="13.235" iyz="0"
     izz="9.655"
+    color="yellow"
     />
-  <xacro:m_joint name="$base_link_world" type="revolute"
+  <xacro:m_joint type="fixed"
          axis_xyz="0 0 1"
          origin_rpy="0 0 0" origin_xyz="0 0 0.0"
          parent="world" child="base_link"
          limit_e="1000" limit_l="0" limit_u="0.5" limit_v="0.5" />
+  <xacro:m_link_mesh
+    name="link1"
+    origin_xyz="0.0 0.0 0.0"
+    origin_rpy="0.0 0.0 0.0"
+    meshfile="package://rjje_arm/meshes/motor_and_frame.stl"
+    meshscale="1 1 1"
+    mass="157.633"
+    ixx="13.235" ixy="0" ixz="0"
+    iyy="13.235" iyz="0"
+    izz="9.655"
+    color="dark_green"
+    />
+  <xacro:m_joint type="fixed"
+     axis_xyz="0 0 1"
+     origin_rpy="0 0 0" origin_xyz="3.45 4.2 4.0"
+     parent="base_link" child="link1"
+     limit_e="1000" limit_l="0" limit_u="0.5" limit_v="0.5" />
+  <xacro:m_link_mesh
+    name="bracket_1"
+    origin_xyz="0.0 0.0 0.0"
+    origin_rpy="0.0 0.0 3.14"
+    meshfile="package://rjje_arm/meshes/thin_bracket.stl"
+    meshscale="1 1 1"
+    mass="157.633"
+    ixx="13.235" ixy="0" ixz="0"
+    iyy="13.235" iyz="0"
+    izz="9.655"
+    color="blue"
+    />
+  <xacro:m_joint type="revolute"
+   axis_xyz="0 0 1"
+   origin_rpy="0 0 0" origin_xyz="0 0 5.3"
+   parent="link1" child="bracket_1"
+   limit_e="1000" limit_l="-1.57" limit_u="1.57" limit_v="0.5" />
 </robot>

File: Fun_Projects/RJJE_Arm/rjje_arm_ws/src/rjje_arm/urdf/rjje_arm.xacro.urdf (robot description, URDF)
Before this commit: robot rjje_arm, 2 links, 1 joints
Links:
- added link bracket_1, mass 157.633; collision mesh filename=package://rjje_arm/meshes/thin_bracket.stl scale=1 1 1; visual mesh filename=package://rjje_arm/meshes/thin_bracket.stl scale=1 1 1
- added link link1, mass 157.633; collision mesh filename=package://rjje_arm/meshes/motor_and_frame.stl scale=1 1 1; visual mesh filename=package://rjje_arm/meshes/motor_and_frame.stl scale=1 1 1
- link base_link: geometry collision mesh filename=package://rjje_arm/meshes/base.stl scale=1 1 1; visual mesh filename=package://rjje_arm/meshes/base.stl scale=1 1 1
Joints:
- removed joint $base_link_world
- added joint base_link_link1: type fixed, parent base_link, child link1, origin xyz=3.45 4.2 4.0 rpy=0 0 0, axis 0 0 1, limit lower=0 upper=0.5 effort=1000 velocity=0.5
- added joint link1_bracket_1: type revolute, parent link1, child bracket_1, origin xyz=0 0 5.3 rpy=0 0 0, axis 0 0 1, limit lower=-1.57 upper=1.57 effort=1000 velocity=0.5
- added joint world_base_link: type fixed, parent world, child base_link, origin xyz=0 0 0.0 rpy=0 0 0, axis 0 0 1, limit lower=0 upper=0.5 effort=1000 velocity=0.5

Commit message: 3d model works!

File: Fun_Projects/RJJE_Arm/rjje_arm_ws/src/rjje_arm/urdf/definitions.xacro (robot description, xacro)
@@ -3,4 +3,7 @@
   <material name="blue">
     <color rgba="0 0 0.8 1"/>
+  </material>
+  <material name="pink">
+    <color rgba="1.0 0.71 0.76 1.0"/>
   </material>
   <material name="yellow">
@@ -41,3 +44,34 @@
     </joint>
   </xacro:macro>
+  <xacro:macro name="m_mimic_joint" params="joint_parent joint_child type axis_xyz origin_rpy origin_xyz parent child limit_e limit_l limit_u limit_v multiplier offset">
+    <joint name="${parent}_${child}" type="${type}">
+      <axis xyz="${axis_xyz}"/>
+      <limit effort="${limit_e}" lower="${limit_l}" upper="${limit_u}" velocity="${limit_v}" />
+      <origin rpy="${origin_rpy}" xyz="${origin_xyz}"/>
+      <parent link="${parent}" />
+      <child link="${child}"/>
+      <mimic joint="${joint_parent}_${joint_child}" multiplier="${multiplier}" offset="${offset}"/>
+    </joint>
+  </xacro:macro>
+  <xacro:macro name="m_fake_link" params="name color origin_xyz origin_rpy length radius">
+    <link name="${name}">
+      <visual>
+        <origin xyz="${origin_xyz}" rpy="${origin_rpy}"/>
+        <geometry>
+            <cylinder length="${length}" radius="${radius}"/>
+         </geometry>
+         <material name="${color}"/>
+      </visual>
+      <collision>
+          <origin xyz="${origin_xyz}" rpy="${origin_rpy}"/>
+          <geometry>
+              <cylinder length="${length}" radius="${radius}"/>
+          </geometry>
+      </collision>
+      <inertial>
+          <mass value="0.1" />
+          <inertia ixx="0.03" iyy="0.03" izz="0.03" ixy="0.0" ixz="0.0" iyz="0.0" />
+      </inertial>
+    </link>
+  </xacro:macro>
 </robot>

File: Fun_Projects/RJJE_Arm/rjje_arm_ws/src/rjje_arm/urdf/rjje_arm.xacro (robot description, xacro)
@@ -18,8 +18,8 @@
     />
   <xacro:m_joint type="fixed"
-         axis_xyz="0 0 1"
-         origin_rpy="0 0 0" origin_xyz="0 0 0.0"
-         parent="world" child="base_link"
-         limit_e="1000" limit_l="0" limit_u="0.5" limit_v="0.5" />
+    axis_xyz="0 0 1"
+    origin_rpy="0 0 0" origin_xyz="0 0 0.0"
+    parent="world" child="base_link"
+    limit_e="1000" limit_l="0" limit_u="0.5" limit_v="0.5" />
   <xacro:m_link_mesh
     name="link1"
@@ -35,8 +35,8 @@
     />
   <xacro:m_joint type="fixed"
-     axis_xyz="0 0 1"
-     origin_rpy="0 0 0" origin_xyz="3.45 4.2 4.0"
-     parent="base_link" child="link1"
-     limit_e="1000" limit_l="0" limit_u="0.5" limit_v="0.5" />
+    axis_xyz="0 0 1"
+    origin_rpy="0 0 0" origin_xyz="3.45 4.2 4.0"
+    parent="base_link" child="link1"
+    limit_e="1000" limit_l="0" limit_u="0.5" limit_v="0.5" />
   <xacro:m_link_mesh
     name="bracket_1"
@@ -52,7 +52,187 @@
     />
   <xacro:m_joint type="revolute"
-   axis_xyz="0 0 1"
-   origin_rpy="0 0 0" origin_xyz="0 0 5.3"
-   parent="link1" child="bracket_1"
-   limit_e="1000" limit_l="-1.57" limit_u="1.57" limit_v="0.5" />
+    axis_xyz="0 0 1"
+    origin_rpy="0 0 0" origin_xyz="0 0 5.3"
+    parent="link1" child="bracket_1"
+    limit_e="1000" limit_l="-1.57" limit_u="1.57" limit_v="0.5" />
+  <xacro:m_link_mesh
+    name="link_2"
+    origin_xyz="0.0 0.0 0.0"
+    origin_rpy="0.0 0.0 0.0"
+    meshfile="package://rjje_arm/meshes/motor_and_frame.stl"
+    meshscale="1 1 1"
+    mass="157.633"
+    ixx="13.235" ixy="0" ixz="0"
+    iyy="13.235" iyz="0"
+    izz="9.655"
+    color="dark_green"
+    />
+  <xacro:m_joint type="fixed"
+    axis_xyz="0 0 1"
+    origin_xyz="2.2 0.0 1.4" origin_rpy="1.57 0.0 -1.57"
+    parent="bracket_1" child="link_2"
+    limit_e="1000" limit_l="-1.57" limit_u="1.57" limit_v="0.5" />
+  <xacro:m_link_mesh
+    name="bracket_2_1"
+    origin_xyz="0.0 0.0 0.0"
+    origin_rpy="0.0 0.0 0.0"
+    meshfile="package://rjje_arm/meshes/thin_bracket.stl"
+    meshscale="1 1 1"
+    mass="157.633"
+    ixx="13.235" ixy="0" ixz="0"
+    iyy="13.235" iyz="0"
+    izz="9.655"
+    color="blue"
+    />
+  <xacro:m_joint type="revolute"
+    axis_xyz="0 0 1"
+    origin_xyz="0.0 0.0 5.3" origin_rpy="0.0 0.0 0.0"
+    parent="link_2" child="bracket_2_1"
+    limit_e="1000" limit_l="-1.57" limit_u="1.57" limit_v="0.5" />
+  <xacro:m_link_mesh
+    name="bracket_2_2"
+    origin_xyz="0.0 0.0 0.0"
+    origin_rpy="0.0 0.0 0.0"
+    meshfile="package://rjje_arm/meshes/thin_bracket.stl"
+    meshscale="1 1 1"
+    mass="157.633"
+    ixx="13.235" ixy="0" ixz="0"
+    iyy="13.235" iyz="0"
+    izz="9.655"
+    color="blue"
+    />
+  <xacro:m_joint type="fixed"
+    axis_xyz="0 0 1"
+    origin_xyz="0.0 10.5 0.0" origin_rpy="0.0 0.0 3.14"
+    parent="bracket_2_1" child="bracket_2_2"
+    limit_e="1000" limit_l="-1.57" limit_u="1.57" limit_v="0.5" />
+  <xacro:m_link_mesh
+    name="link_3"
+    origin_xyz="0.0 0.0 0.0"
+    origin_rpy="0.0 0.0 0.0"
+    meshfile="package://rjje_arm/meshes/motor_and_frame.stl"
+    meshscale="1 1 1"
+    mass="157.633"
+    ixx="13.235" ixy="0" ixz="0"
+    iyy="13.235" iyz="0"
+    izz="9.655"
+    color="dark_green"
+    />
+  <xacro:m_joint type="revolute"
+    axis_xyz="0 0 1"
+    origin_xyz="0.0 0.0 -5.3" origin_rpy="0.0 0.0 3.14"
+    parent="bracket_2_2" child="link_3"
+    limit_e="1000" limit_l="-1.57" limit_u="1.57" limit_v="0.5" />
+  <!-- This is a "fake" link that represents attachment to link 3 -->
+  <xacro:m_fake_link
+    name="bracket_3_1"
+    color="pink"
+    origin_xyz="0.0 0.0 0.75"
+    origin_rpy="0.0 0.0 0.0"
+    length="1.5"
+    radius="0.5"
+    />
+  <xacro:m_joint type="fixed"
+    axis_xyz="0 0 1"
+    origin_xyz="4.0 0.0 2.0" origin_rpy="0.0 1.57 0.0"
+    parent="link_3" child="bracket_3_1"
+    limit_e="1000" limit_l="-1.57" limit_u="1.57" limit_v="0.5" />
+  <xacro:m_link_mesh
+    name="bracket_3_2"
+    origin_xyz="0.0 0.0 0.0"
+    origin_rpy="0.0 0.0 0.0"
+    meshfile="package://rjje_arm/meshes/thin_bracket.stl"
+    meshscale="1 1 1"
+    mass="157.633"
+    ixx="13.235" ixy="0" ixz="0"
+    iyy="13.235" iyz="0"
+    izz="9.655"
+    color="blue"
+    />
+  <xacro:m_joint type="fixed"
+    axis_xyz="0 0 1"
+    origin_xyz="-2.65 0.0 6.75" origin_rpy="-1.57 0.0 1.57"
+    parent="bracket_3_1" child="bracket_3_2"
+    limit_e="1000" limit_l="-1.57" limit_u="1.57" limit_v="0.5" />
+  <xacro:m_link_mesh
+    name="link_4"
+    origin_xyz="0.0 0.0 0.0"
+    origin_rpy="0.0 0.0 0.0"
+    meshfile="package://rjje_arm/meshes/motor_and_frame.stl"
+    meshscale="1 1 1"
+    mass="157.633"
+    ixx="13.235" ixy="0" ixz="0"
+    iyy="13.235" iyz="0"
+    izz="9.655"
+    color="dark_green"
+    />
+  <xacro:m_joint type="revolute"
+    axis_xyz="0 0 1"
+    origin_xyz="0.0 0.0 -5.3" origin_rpy="0.0 0.0 -1.57"
+    parent="bracket_3_2" child="link_4"
+    limit_e="1000" limit_l="-1.57" limit_u="0.43" limit_v="0.5" />
+  <xacro:m_link_mesh
+    name="link_5"
+    origin_xyz="0.0 0.0 0.0"
+    origin_rpy="0.0 0.0 0.0"
+    meshfile="package://rjje_arm/meshes/motor_and_frame.stl"
+    meshscale="1 1 1"
+    mass="157.633"
+    ixx="13.235" ixy="0" ixz="0"
+    iyy="13.235" iyz="0"
+    izz="9.655"
+    color="dark_green"
+    />
+  <xacro:m_joint type="fixed"
+    axis_xyz="0 0 1"
+    origin_xyz="0.0 2.4 2.2" origin_rpy="0.0 1.57 0.0"
+    parent="link_4" child="link_5"
+    limit_e="1000" limit_l="-1.57" limit_u="1.57" limit_v="0.5" />
+  <xacro:m_link_mesh
+    name="left_gripper"
+    origin_xyz="0.0 0.0 0.0"
+    origin_rpy="0.0 0.0 0.0"
+    meshfile="package://rjje_arm/meshes/left_gripper.stl"
+    meshscale="1 1 1"
+    mass="157.633"
+    ixx="13.235" ixy="0" ixz="0"
+    iyy="13.235" iyz="0"
+    izz="9.655"
+    color="yellow"
+    />
+  <xacro:m_joint type="revolute"
+    axis_xyz="0 1 0"
+    origin_xyz="0.0 0.0 5.2" origin_rpy="0.0 0.0 0.0"
+    parent="link_5" child="left_gripper"
+    limit_e="1000" limit_l="-0.61" limit_u="0.0" limit_v="0.5" />
+  <xacro:m_link_mesh
+    name="right_gripper"
+    origin_xyz="0.0 0.0 0.0"
+    origin_rpy="0.0 0.0 0.0"
+    meshfile="package://rjje_arm/meshes/right_gripper.stl"
+    meshscale="1 1 1"
+    mass="157.633"
+    ixx="13.235" ixy="0" ixz="0"
+    iyy="13.235" iyz="0"
+    izz="9.655"
+    color="yellow"
+    />
+    <!-- TODO -->
+  <!-- <xacro:m_joint  -->
+  <!--   type="revolute" -->
+  <!--   axis_xyz="0 1 0" -->
+  <!--   origin_xyz="0.0 0.0 5.2" origin_rpy="0.0 0.0 0.0" -->
+  <!--   parent="link_5" child="right_gripper" -->
+  <!--   limit_e="1000" limit_l="0.65" limit_u="&#45;0.15" limit_v="0.5" /> -->
+  <xacro:m_mimic_joint
+    joint_parent="link_5"
+    joint_child="left_gripper"
+    type="revolute"
+    axis_xyz="0 1 0"
+    origin_xyz="0.0 0.0 5.2" origin_rpy="0.0 0.0 0.0"
+    parent="link_5" child="right_gripper"
+    limit_e="1000" limit_l="0.61" limit_u="0.0" limit_v="0.5"
+    multiplier="-1"
+    offset="0"
+    />
 </robot>

File: Fun_Projects/RJJE_Arm/rjje_arm_ws/src/rjje_arm/urdf/rjje_arm.xacro.urdf (robot description, URDF)
Before this commit: robot rjje_arm, 4 links, 3 joints
Links:
- added link bracket_2_1, mass 157.633; collision mesh filename=package://rjje_arm/meshes/thin_bracket.stl scale=1 1 1; visual mesh filename=package://rjje_arm/meshes/thin_bracket.stl scale=1 1 1
- added link bracket_2_2, mass 157.633; collision mesh filename=package://rjje_arm/meshes/thin_bracket.stl scale=1 1 1; visual mesh filename=package://rjje_arm/meshes/thin_bracket.stl scale=1 1 1
- added link bracket_3_1, mass 0.1; collision cylinder length=1.5 radius=0.5; visual cylinder length=1.5 radius=0.5
- added link bracket_3_2, mass 157.633; collision mesh filename=package://rjje_arm/meshes/thin_bracket.stl scale=1 1 1; visual mesh filename=package://rjje_arm/meshes/thin_bracket.stl scale=1 1 1
- added link left_gripper, mass 157.633; collision mesh filename=package://rjje_arm/meshes/left_gripper.stl scale=1 1 1; visual mesh filename=package://rjje_arm/meshes/left_gripper.stl scale=1 1 1
- added link link_2, mass 157.633; collision mesh filename=package://rjje_arm/meshes/motor_and_frame.stl scale=1 1 1; visual mesh filename=package://rjje_arm/meshes/motor_and_frame.stl scale=1 1 1
- added link link_3, mass 157.633; collision mesh filename=package://rjje_arm/meshes/motor_and_frame.stl scale=1 1 1; visual mesh filename=package://rjje_arm/meshes/motor_and_frame.stl scale=1 1 1
- added link link_4, mass 157.633; collision mesh filename=package://rjje_arm/meshes/motor_and_frame.stl scale=1 1 1; visual mesh filename=package://rjje_arm/meshes/motor_and_frame.stl scale=1 1 1
- added link link_5, mass 157.633; collision mesh filename=package://rjje_arm/meshes/motor_and_frame.stl scale=1 1 1; visual mesh filename=package://rjje_arm/meshes/motor_and_frame.stl scale=1 1 1
- added link right_gripper, mass 157.633; collision mesh filename=package://rjje_arm/meshes/right_gripper.stl scale=1 1 1; visual mesh filename=package://rjje_arm/meshes/right_gripper.stl scale=1 1 1
Joints:
- added joint bracket_1_link_2: type fixed, parent bracket_1, child link_2, origin xyz=2.2 0.0 1.4 rpy=1.57 0.0 -1.57, axis 0 0 1, limit lower=-1.57 upper=1.57 effort=1000 velocity=0.5
- added joint bracket_2_1_bracket_2_2: type fixed, parent bracket_2_1, child bracket_2_2, origin xyz=0.0 10.5 0.0 rpy=0.0 0.0 3.14, axis 0 0 1, limit lower=-1.57 upper=1.57 effort=1000 velocity=0.5
- added joint bracket_2_2_link_3: type revolute, parent bracket_2_2, child link_3, origin xyz=0.0 0.0 -5.3 rpy=0.0 0.0 3.14, axis 0 0 1, limit lower=-1.57 upper=1.57 effort=1000 velocity=0.5
- added joint bracket_3_1_bracket_3_2: type fixed, parent bracket_3_1, child bracket_3_2, origin xyz=-2.65 0.0 6.75 rpy=-1.57 0.0 1.57, axis 0 0 1, limit lower=-1.57 upper=1.57 effort=1000 velocity=0.5
- added joint bracket_3_2_link_4: type revolute, parent bracket_3_2, child link_4, origin xyz=0.0 0.0 -5.3 rpy=0.0 0.0 -1.57, axis 0 0 1, limit lower=-1.57 upper=0.43 effort=1000 velocity=0.5
- added joint link_2_bracket_2_1: type revolute, parent link_2, child bracket_2_1, origin xyz=0.0 0.0 5.3 rpy=0.0 0.0 0.0, axis 0 0 1, limit lower=-1.57 upper=1.57 effort=1000 velocity=0.5
- added joint link_3_bracket_3_1: type fixed, parent link_3, child bracket_3_1, origin xyz=4.0 0.0 2.0 rpy=0.0 1.57 0.0, axis 0 0 1, limit lower=-1.57 upper=1.57 effort=1000 velocity=0.5
- added joint link_4_link_5: type fixed, parent link_4, child link_5, origin xyz=0.0 2.4 2.2 rpy=0.0 1.57 0.0, axis 0 0 1, limit lower=-1.57 upper=1.57 effort=1000 velocity=0.5
- added joint link_5_left_gripper: type revolute, parent link_5, child left_gripper, origin xyz=0.0 0.0 5.2 rpy=0.0 0.0 0.0, axis 0 1 0, limit lower=-0.61 upper=0.0 effort=1000 velocity=0.5
- added joint link_5_right_gripper: type revolute, parent link_5, child right_gripper, origin xyz=0.0 0.0 5.2 rpy=0.0 0.0 0.0, axis 0 1 0, limit lower=0.61 upper=0.0 effort=1000 velocity=0.5, mimic joint=link_5_left_gripper multiplier=-1 offset=0
