Commit message: cleaned up, modified project notes

File: Fun_Projects/RJJE_Arm/rjje_arm_ws/src/rjje_arm/urdf/rjje_arm.xacro (robot description, xacro)
@@ -17,4 +17,7 @@
     color="yellow"
     />
+  <gazebo reference="base_link">
+    <material>Gazebo/Yellow</material>
+  </gazebo>
   <xacro:m_joint type="fixed"
     axis_xyz="0 0 1"
@@ -55,5 +58,5 @@
     origin_rpy="0 0 0" origin_xyz="0 0 5.3"
     parent="link1" child="bracket_1"
-    limit_e="1000" limit_l="-1.57" limit_u="1.57" limit_v="0.5" />
+    limit_e="1000" limit_l="-1.57" limit_u="1.57" limit_v="1.5" />
   <xacro:m_link_mesh
     name="link_2"
@@ -89,5 +92,5 @@
     origin_xyz="0.0 0.0 5.3" origin_rpy="0.0 0.0 0.0"
     parent="link_2" child="bracket_2_1"
-    limit_e="1000" limit_l="-1.57" limit_u="1.57" limit_v="0.5" />
+    limit_e="1000" limit_l="-1.57" limit_u="1.57" limit_v="1.5" />
   <xacro:m_link_mesh
     name="bracket_2_2"
@@ -123,5 +126,5 @@
     origin_xyz="0.0 0.0 -5.3" origin_rpy="0.0 0.0 3.14"
     parent="bracket_2_2" child="link_3"
-    limit_e="1000" limit_l="-1.57" limit_u="1.57" limit_v="0.5" />
+    limit_e="1000" limit_l="-1.57" limit_u="1.57" limit_v="1.5" />
   <!-- This is a "fake" link that represents attachment to link 3 -->
   <xacro:m_fake_link
@@ -171,5 +174,5 @@
     origin_xyz="0.0 0.0 -5.3" origin_rpy="0.0 0.0 -1.57"
     parent="bracket_3_2" child="link_4"
-    limit_e="1000" limit_l="-1.57" limit_u="0.43" limit_v="0.5" />
+    limit_e="1000" limit_l="-1.57" limit_u="0.43" limit_v="1.5" />
   <xacro:m_link_mesh
     name="link_5"
@@ -190,4 +193,21 @@
     limit_e="1000" limit_l="-1.57" limit_u="1.57" limit_v="0.5" />
   <xacro:m_link_mesh
+    name="link_6"
+    origin_xyz="0.0 0.0 0.0"
+    origin_rpy="0.0 0.0 0.0"
+    meshfile="package://rjje_arm/meshes/motor_and_frame.stl"
+    meshscale="0 0 0"
+    mass="157.633"
+    ixx="13.235" ixy="0" ixz="0"
+    iyy="13.235" iyz="0"
+    izz="9.655"
+    color="dark_green"
+    />
+  <xacro:m_joint type="revolute"
+    axis_xyz="0 0 1"
+    origin_xyz="0.0 0.0 0.0" origin_rpy="0.0 0.0 0.0"
+    parent="link_5" child="link_6"
+    limit_e="1000" limit_l="-1.57" limit_u="1.57" limit_v="1.5" />
+  <xacro:m_link_mesh
     name="left_gripper"
     origin_xyz="0.0 0.0 0.0"
@@ -204,6 +224,6 @@
     axis_xyz="0 1 0"
     origin_xyz="0.0 0.0 5.2" origin_rpy="0.0 0.0 0.0"
-    parent="link_5" child="left_gripper"
-    limit_e="1000" limit_l="-0.61" limit_u="0.0" limit_v="0.5" />
+    parent="link_6" child="left_gripper"
+    limit_e="1000" limit_l="-0.61" limit_u="0.0" limit_v="1.5" />
   <xacro:m_link_mesh
     name="right_gripper"
@@ -219,11 +239,11 @@
     />
   <xacro:m_mimic_joint
-    joint_parent="link_5"
+    joint_parent="link_6"
     joint_child="left_gripper"
     type="revolute"
     axis_xyz="0 1 0"
     origin_xyz="0.0 0.0 5.2" origin_rpy="0.0 0.0 0.0"
-    parent="link_5" child="right_gripper"
-    limit_e="1000" limit_l="0.61" limit_u="0.0" limit_v="0.5"
+    parent="link_6" child="right_gripper"
+    limit_e="1000" limit_l="0.61" limit_u="0.0" limit_v="1.5"
     multiplier="-1"
     offset="0"

File: Fun_Projects/RJJE_Arm/rjje_arm_ws/src/rjje_arm/urdf/rjje_arm.xacro.urdf (robot description, URDF)
Before this commit: robot rjje_arm, 14 links, 13 joints
Links:
- added link link_6, mass 157.633; collision mesh filename=package://rjje_arm/meshes/motor_and_frame.stl scale=0 0 0; visual mesh filename=package://rjje_arm/meshes/motor_and_frame.stl scale=0 0 0
Joints:
- removed joint link_5_left_gripper
- removed joint link_5_right_gripper
- added joint link_5_link_6: type revolute, parent link_5, child link_6, origin xyz=0.0 0.0 0.0 rpy=0.0 0.0 0.0, axis 0 0 1, limit lower=-1.57 upper=1.57 effort=1000 velocity=1.5
- added joint link_6_left_gripper: type revolute, parent link_6, child left_gripper, origin xyz=0.0 0.0 5.2 rpy=0.0 0.0 0.0, axis 0 1 0, limit lower=-0.61 upper=0.0 effort=1000 velocity=1.5
- added joint link_6_right_gripper: type revolute, parent link_6, child right_gripper, origin xyz=0.0 0.0 5.2 rpy=0.0 0.0 0.0, axis 0 1 0, limit lower=0.61 upper=0.0 effort=1000 velocity=1.5, mimic joint=link_6_left_gripper multiplier=-1 offset=0
- joint bracket_2_2_link_3: limit lower=-1.57 upper=1.57 effort=1000 velocity=0.5 -> lower=-1.57 upper=1.57 effort=1000 velocity=1.5
- joint bracket_3_2_link_4: limit lower=-1.57 upper=0.43 effort=1000 velocity=0.5 -> lower=-1.57 upper=0.43 effort=1000 velocity=1.5
- joint link1_bracket_1: limit lower=-1.57 upper=1.57 effort=1000 velocity=0.5 -> lower=-1.57 upper=1.57 effort=1000 velocity=1.5
- joint link_2_bracket_2_1: limit lower=-1.57 upper=1.57 effort=1000 velocity=0.5 -> lower=-1.57 upper=1.57 effort=1000 velocity=1.5
